Commit message: fix waypoint loading

File: src/myrobot_description/urdf/robot/my_robot_homemade.xacro (robot description, xacro)
@@ -3,6 +3,6 @@
   <xacro:include filename="inertial_macros.xacro"/>
   <xacro:property name="base_length" value="0.20" />
-  <xacro:property name="base_width" value="0.34" />
-  <xacro:property name="base_height" value="0.30" />
+  <xacro:property name="base_width" value="0.31" />
+  <xacro:property name="base_height" value="0.20" />
   <xacro:property name="base_mass" value="3.0" />
   <xacro:property name="wheel_mass" value="0.3" />

File: src/myrobot_description/urdf/robot/myrobot_gazebo.xacro (robot description, xacro)
@@ -3,25 +3,25 @@
   <!-- Wheels -->
 <gazebo reference="left_wheel_link">
-  <mu1>0.8</mu1>
-  <mu2>0.8</mu2>
+  <mu1>200.0</mu1>
+  <mu2>100.0</mu2>
   <kp>1000000.0</kp>
-  <kd>10.0</kd>
-  <minDepth>0.001</minDepth>
-  <maxVel>1.0</maxVel>
+  <kd>100.0</kd>
+  <minDepth>0.0</minDepth>
+  <maxVel>0.1</maxVel>
   <fdir1>1 0 0</fdir1>
 </gazebo>
 <gazebo reference="right_wheel_link">
-  <mu1>0.8</mu1>
-  <mu2>0.8</mu2>
+  <mu1>200.0</mu1>
+  <mu2>100.0</mu2>
   <kp>1000000.0</kp>
-  <kd>10.0</kd>
-  <minDepth>0.001</minDepth>
-  <maxVel>1.0</maxVel>
+  <kd>100.0</kd>
+  <minDepth>0.0</minDepth>
+  <maxVel>0.1</maxVel>
   <fdir1>1 0 0</fdir1>
 </gazebo>
   <!-- Caster Wheels -->
   <gazebo reference="rear_caster_wheel_link">
-    <mu1>0.1</mu1>
-    <mu2>0.1</mu2>
+    <mu1>0.0</mu1>
+    <mu2>0.0</mu2>
     <kp>1000000.0</kp>
     <kd>100.0</kd>
@@ -30,6 +30,6 @@
   </gazebo>
   <gazebo reference="front_caster_wheel_link">
-    <mu1>0.1</mu1>
-    <mu2>0.1</mu2>
+    <mu1>0.0</mu1>
+    <mu2>0.0</mu2>
     <kp>1000000.0</kp>
     <kd>100.0</kd>
@@ -45,4 +45,12 @@
       <plugin filename="gz-sim-sensors-system" name="gz::sim::systems::Sensors">
         <render_engine>ogre2</render_engine>
+      </plugin>
+      <!-- Ground Truth Odometry Publisher (from Gazebo physics, not from wheel encoders) -->
+      <plugin filename="gz-sim-odometry-publisher-system" name="gz::sim::systems::OdometryPublisher">
+        <link_name>base_footprint</link_name>
+        <odom_frame>odom</odom_frame>
+        <body_frame>base_footprint</body_frame>
+        <odom_publish_frequency>50</odom_publish_frequency>
+        <odom_topic>ground_truth/odom</odom_topic>
       </plugin>
   </gazebo>

File: src/myrobot_description/urdf/robot/robot_ros2_control.xacro (robot description, xacro)
@@ -19,6 +19,6 @@
         <joint name="right_wheel_joint">
             <command_interface name="velocity">
-                <param name="min">-1</param>
-                <param name="max">1</param>
+                <param name="min">-10</param>
+                <param name="max">10</param>
             </command_interface>
             <state_interface name="position" />
@@ -27,6 +27,6 @@
         <joint name="left_wheel_joint">
             <command_interface name="velocity">
-                <param name="min">-1</param>
-                <param name="max">1</param>
+                <param name="min">-10</param>
+                <param name="max">10</param>
             </command_interface>
             <state_interface name="position" />
